Commit message: 新增六足控制器和雅可比计算，更新URDF模型路径

File: urdf/hexapod_collision.urdf (robot description, URDF)
Before this commit: robot hexapod_robot, 25 links, 24 joints
Links:
- link base_link: geometry collision cylinder length=0.121 radius=0.097; visual mesh filename=../meshes/body_link.STL
- link lb_ankle_link: geometry collision box size=0.130 0.022 0.022; visual mesh filename=../meshes/ankle_link.STL
- link lb_knee_link: geometry collision box size=0.07745 0.022 0.022; visual mesh filename=../meshes/knee_link.STL
- link lb_thigh_link: geometry collision box size=0.05236 0.025 0.025; visual mesh filename=../meshes/thigh_link.STL
- link lf_ankle_link: geometry collision box size=0.130 0.022 0.022; visual mesh filename=../meshes/ankle_link.STL
- link lf_knee_link: geometry collision box size=0.07745 0.022 0.022; visual mesh filename=../meshes/knee_link.STL
- link lf_thigh_link: geometry collision box size=0.05236 0.025 0.025; visual mesh filename=../meshes/thigh_link.STL
- link lm_ankle_link: geometry collision box size=0.130 0.022 0.022; visual mesh filename=../meshes/ankle_link.STL
- link lm_knee_link: geometry collision box size=0.07745 0.022 0.022; visual mesh filename=../meshes/knee_link.STL
- link lm_thigh_link: geometry collision box size=0.05236 0.025 0.025; visual mesh filename=../meshes/thigh_link.STL
- link rb_ankle_link: geometry collision box size=0.130 0.022 0.022; visual mesh filename=../meshes/ankle_link.STL
- link rb_knee_link: geometry collision box size=0.07745 0.022 0.022; visual mesh filename=../meshes/knee_link.STL
- link rb_thigh_link: geometry collision box size=0.05236 0.025 0.025; visual mesh filename=../meshes/thigh_link.STL
- link rf_ankle_link: geometry collision box size=0.130 0.022 0.022; visual mesh filename=../meshes/ankle_link.STL
- link rf_knee_link: geometry collision box size=0.07745 0.022 0.022; visual mesh filename=../meshes/knee_link.STL
- link rf_thigh_link: geometry collision box size=0.05236 0.025 0.025; visual mesh filename=../meshes/thigh_link.STL
- link rm_ankle_link: geometry collision box size=0.130 0.022 0.022; visual mesh filename=../meshes/ankle_link.STL
- link rm_knee_link: geometry collision box size=0.07745 0.022 0.022; visual mesh filename=../meshes/knee_link.STL
- link rm_thigh_link: geometry collision box size=0.05236 0.025 0.025; visual mesh filename=../meshes/thigh_link.STL

File: urdf/hexapodurdf.urdf.xacro (robot description, xacro)
@@ -3,6 +3,4 @@
   <material name="white"><color rgba="1 1 1 1"/></material>
   <material name="foot_black"><color rgba="0.02 0.02 0.02 1"/></material>
-  <!-- Package / mesh paths -->
-  <xacro:property name="mesh_pkg" value="hexapod_robot"/>
   <!-- Actuator / joint limits -->
   <xacro:property name="servo_effort" value="1.2"/>
@@ -43,5 +41,5 @@
       <origin xyz="0 0 0" rpy="0 0 0"/>
       <geometry>
-        <mesh filename="package://${mesh_pkg}/meshes/${mesh_file}"/>
+        <mesh filename="../meshes/${mesh_file}"/>
       </geometry>
       <material name="white">

File: urdf/抓取机器人export_urdf.SLDASM.urdf (robot description, URDF)
Before this commit: robot 抓取机器人export_urdf.SLDASM, 19 links, 18 joints
Links:
- link base_link: geometry collision mesh filename=../meshes/body_link.STL; visual mesh filename=../meshes/body_link.STL
- link lb_ankle_Link: geometry collision mesh filename=../meshes/ankle_link.STL; visual mesh filename=../meshes/ankle_link.STL
- link lb_knee_Link: geometry collision mesh filename=../meshes/knee_link.STL; visual mesh filename=../meshes/knee_link.STL
- link lb_thigh_Link: geometry collision mesh filename=../meshes/thigh_link.STL; visual mesh filename=../meshes/thigh_link.STL
- link lf_ankle_Link: geometry collision mesh filename=../meshes/ankle_link.STL; visual mesh filename=../meshes/ankle_link.STL
- link lf_knee_Link: geometry collision mesh filename=../meshes/knee_link.STL; visual mesh filename=../meshes/knee_link.STL
- link lf_thigh_Link: geometry collision mesh filename=../meshes/thigh_link.STL; visual mesh filename=../meshes/thigh_link.STL
- link lm_ankle_Link: geometry collision mesh filename=../meshes/ankle_link.STL; visual mesh filename=../meshes/ankle_link.STL
- link lm_knee_Link: geometry collision mesh filename=../meshes/knee_link.STL; visual mesh filename=../meshes/knee_link.STL
- link lm_thigh_Link: geometry collision mesh filename=../meshes/thigh_link.STL; visual mesh filename=../meshes/thigh_link.STL
- link rb_ankle_Link: geometry collision mesh filename=../meshes/ankle_link.STL; visual mesh filename=../meshes/ankle_link.STL
- link rb_knee_Link: geometry collision mesh filename=../meshes/knee_link.STL; visual mesh filename=../meshes/knee_link.STL
- link rb_thigh_Link: geometry collision mesh filename=../meshes/thigh_link.STL; visual mesh filename=../meshes/thigh_link.STL
- link rf_ankle_Link: geometry collision mesh filename=../meshes/ankle_link.STL; visual mesh filename=../meshes/ankle_link.STL
- link rf_knee_Link: geometry collision mesh filename=../meshes/knee_link.STL; visual mesh filename=../meshes/knee_link.STL
- link rf_thigh_Link: geometry collision mesh filename=../meshes/thigh_link.STL; visual mesh filename=../meshes/thigh_link.STL
- link rm_ankle_Link: geometry collision mesh filename=../meshes/ankle_link.STL; visual mesh filename=../meshes/ankle_link.STL
- link rm_knee_Link: geometry collision mesh filename=../meshes/knee_link.STL; visual mesh filename=../meshes/knee_link.STL
- link rm_thigh_Link: geometry collision mesh filename=../meshes/thigh_link.STL; visual mesh filename=../meshes/thigh_link.STL
