Commit message: Refactor control script and update URDF joint limits
- Modified `run_control_isaacgym.py` to include joystick control for motion enabling, resetting to stand, and smooth command handling.
- Adjusted the robot's base height during initialization and removed unnecessary velocity control calculations.
- Updated the URDF file to change the joint limits for ankle joints from [-1.745, 1.745] to [-2.094, 2.094] to allow for greater range of motion.

File: urdf/hexapod_isaacgym_view.urdf (robot description, URDF)
Before this commit: robot hexapod_robot, 25 links, 24 joints
Joints:
- joint lb_ankle_joint: limit lower=-1.745 upper=1.745 effort=1.2 velocity=4.0 -> lower=-2.094 upper=2.094 effort=1.2 velocity=4.0
- joint lf_ankle_joint: limit lower=-1.745 upper=1.745 effort=1.2 velocity=4.0 -> lower=-2.094 upper=2.094 effort=1.2 velocity=4.0
- joint lm_ankle_joint: limit lower=-1.745 upper=1.745 effort=1.2 velocity=4.0 -> lower=-2.094 upper=2.094 effort=1.2 velocity=4.0
- joint rb_ankle_joint: limit lower=-1.745 upper=1.745 effort=1.2 velocity=4.0 -> lower=-2.094 upper=2.094 effort=1.2 velocity=4.0
- joint rf_ankle_joint: limit lower=-1.745 upper=1.745 effort=1.2 velocity=4.0 -> lower=-2.094 upper=2.094 effort=1.2 velocity=4.0
- joint rm_ankle_joint: limit lower=-1.745 upper=1.745 effort=1.2 velocity=4.0 -> lower=-2.094 upper=2.094 effort=1.2 velocity=4.0
