Commit message: Add validation script for climb preview and update descriptions
- Introduced `validate_climb_preview.py` for integrity checks on the Isaac-only compact plan.
- Updated package descriptions in `package.xml` files for `grasp_hexapod_description` and `grasp_hexapod_servo` to Chinese.
- Adjusted collision box sizes in URDF files for `hexapod_collision.urdf` and `hexapod_isaacgym_view.urdf`.
- Enhanced documentation in `hiwonder_servo_controller.py` with detailed parameter descriptions and method explanations.
- Cleaned up exception handling in `hiwonder_servo_controller.py` and `servo.py`.

File: src/grasp_hexapod_description/urdf/hexapod_collision.urdf (robot description, URDF)
Before this commit: robot hexapod_robot, 25 links, 24 joints
Links:
- link lb_ankle_link: geometry collision box size=0.130 0.006 0.006; visual mesh filename=../meshes/ankle_link.STL
- link lf_ankle_link: geometry collision box size=0.130 0.006 0.006; visual mesh filename=../meshes/ankle_link.STL
- link lm_ankle_link: geometry collision box size=0.130 0.006 0.006; visual mesh filename=../meshes/ankle_link.STL
- link rb_ankle_link: geometry collision box size=0.130 0.006 0.006; visual mesh filename=../meshes/ankle_link.STL
- link rf_ankle_link: geometry collision box size=0.130 0.006 0.006; visual mesh filename=../meshes/ankle_link.STL
- link rm_ankle_link: geometry collision box size=0.130 0.006 0.006; visual mesh filename=../meshes/ankle_link.STL

File: src/grasp_hexapod_description/urdf/hexapod_isaacgym_view.urdf (robot description, URDF)
Before this commit: robot hexapod_robot, 25 links, 24 joints
Links:
- link lb_ankle_link: geometry collision box size=0.130 0.006 0.006; visual mesh filename=../meshes/ankle_link.STL
- link lf_ankle_link: geometry collision box size=0.130 0.006 0.006; visual mesh filename=../meshes/ankle_link.STL
- link lm_ankle_link: geometry collision box size=0.130 0.006 0.006; visual mesh filename=../meshes/ankle_link.STL
- link rb_ankle_link: geometry collision box size=0.130 0.006 0.006; visual mesh filename=../meshes/ankle_link.STL
- link rf_ankle_link: geometry collision box size=0.130 0.006 0.006; visual mesh filename=../meshes/ankle_link.STL
- link rm_ankle_link: geometry collision box size=0.130 0.006 0.006; visual mesh filename=../meshes/ankle_link.STL
