Commit message: Add SDK components for hardware control and reference documents
- Introduced new SDK modules for button, buzzer, encoder motor, IMU, LED, PWM servo, and Hiwonder servo control.
- Added initialization and control functions for each hardware component.
- Included reference PDF documents for various hardware configurations.
- Implemented GPIO setup and handling for button and LED functionalities.
- Established I2C communication for encoder motor and IMU data retrieval.
- Created methods for servo position control and feedback.

File: src/grasp_hexapod_description/urdf/grasp_hexapod.urdf (robot description, URDF)
Before this commit: robot grasp_hexapod, 19 links, 18 joints
Joints:
- joint lb_ankle_joint: limit lower=-1.745 upper=1.745 effort=1.2 velocity=4 -> lower=-2.094 upper=2.094 effort=1.2 velocity=4
- joint lf_ankle_joint: limit lower=-1.745 upper=1.745 effort=1.2 velocity=4 -> lower=-2.094 upper=2.094 effort=1.2 velocity=4
- joint lm_ankle_joint: limit lower=-1.745 upper=1.745 effort=1.2 velocity=4 -> lower=-2.094 upper=2.094 effort=1.2 velocity=4
- joint rb_ankle_joint: limit lower=-1.745 upper=1.745 effort=1.2 velocity=4 -> lower=-2.094 upper=2.094 effort=1.2 velocity=4
- joint rf_ankle_joint: limit lower=-1.745 upper=1.745 effort=1.2 velocity=4 -> lower=-2.094 upper=2.094 effort=1.2 velocity=4
- joint rm_ankle_joint: limit lower=-1.745 upper=1.745 effort=1.2 velocity=4 -> lower=-2.094 upper=2.094 effort=1.2 velocity=4

File: src/grasp_hexapod_description/urdf/hexapodurdf.urdf.xacro (robot description, xacro)
@@ -8,6 +8,6 @@
   <xacro:property name="knee_lower" value="-2.094"/>
   <xacro:property name="knee_upper" value="2.094"/>
-  <xacro:property name="ankle_lower" value="-1.745"/>
-  <xacro:property name="ankle_upper" value="1.745"/>
+  <xacro:property name="ankle_lower" value="-2.094"/>
+  <xacro:property name="ankle_upper" value="2.094"/>
   <!-- Joint geometry -->
   <xacro:property name="thigh_to_knee_x" value="0.05236"/>

Commit message: 阶段性提交

File: src/grasp_hexapod_description/urdf/grasp_hexapod.urdf (robot description, URDF)
Before this commit: robot grasp_hexapod, 19 links, 18 joints
Links:
- link base_link: geometry collision mesh filename=package://grasp_hexapod_description/meshes/body_link.STL; visual mesh filename=package://grasp_hexapod_description/meshes/body_link.STL
- link lb_ankle_Link: geometry collision mesh filename=package://grasp_hexapod_description/meshes/ankle_link.STL; visual mesh filename=package://grasp_hexapod_description/meshes/ankle_link.STL
- link lb_knee_Link: geometry collision mesh filename=package://grasp_hexapod_description/meshes/knee_link.STL; visual mesh filename=package://grasp_hexapod_description/meshes/knee_link.STL
- link lb_thigh_Link: geometry collision mesh filename=package://grasp_hexapod_description/meshes/thigh_link.STL; visual mesh filename=package://grasp_hexapod_description/meshes/thigh_link.STL
- link lf_ankle_Link: geometry collision mesh filename=package://grasp_hexapod_description/meshes/ankle_link.STL; visual mesh filename=package://grasp_hexapod_description/meshes/ankle_link.STL
- link lf_knee_Link: geometry collision mesh filename=package://grasp_hexapod_description/meshes/knee_link.STL; visual mesh filename=package://grasp_hexapod_description/meshes/knee_link.STL
- link lf_thigh_Link: geometry collision mesh filename=package://grasp_hexapod_description/meshes/thigh_link.STL; visual mesh filename=package://grasp_hexapod_description/meshes/thigh_link.STL
- link lm_ankle_Link: geometry collision mesh filename=package://grasp_hexapod_description/meshes/ankle_link.STL; visual mesh filename=package://grasp_hexapod_description/meshes/ankle_link.STL
- link lm_knee_Link: geometry collision mesh filename=package://grasp_hexapod_description/meshes/knee_link.STL; visual mesh filename=package://grasp_hexapod_description/meshes/knee_link.STL
- link lm_thigh_Link: geometry collision mesh filename=package://grasp_hexapod_description/meshes/thigh_link.STL; visual mesh filename=package://grasp_hexapod_description/meshes/thigh_link.STL
- link rb_ankle_Link: geometry collision mesh filename=package://grasp_hexapod_description/meshes/ankle_link.STL; visual mesh filename=package://grasp_hexapod_description/meshes/ankle_link.STL
- link rb_knee_Link: geometry collision mesh filename=package://grasp_hexapod_description/meshes/knee_link.STL; visual mesh filename=package://grasp_hexapod_description/meshes/knee_link.STL
- link rb_thigh_Link: geometry collision mesh filename=package://grasp_hexapod_description/meshes/thigh_link.STL; visual mesh filename=package://grasp_hexapod_description/meshes/thigh_link.STL
- link rf_ankle_Link: geometry collision mesh filename=package://grasp_hexapod_description/meshes/ankle_link.STL; visual mesh filename=package://grasp_hexapod_description/meshes/ankle_link.STL
- link rf_knee_Link: geometry collision mesh filename=package://grasp_hexapod_description/meshes/knee_link.STL; visual mesh filename=package://grasp_hexapod_description/meshes/knee_link.STL
- link rf_thigh_Link: geometry collision mesh filename=package://grasp_hexapod_description/meshes/thigh_link.STL; visual mesh filename=package://grasp_hexapod_description/meshes/thigh_link.STL
- link rm_ankle_Link: geometry collision mesh filename=package://grasp_hexapod_description/meshes/ankle_link.STL; visual mesh filename=package://grasp_hexapod_description/meshes/ankle_link.STL
- link rm_knee_Link: geometry collision mesh filename=package://grasp_hexapod_description/meshes/knee_link.STL; visual mesh filename=package://grasp_hexapod_description/meshes/knee_link.STL
- link rm_thigh_Link: geometry collision mesh filename=package://grasp_hexapod_description/meshes/thigh_link.STL; visual mesh filename=package://grasp_hexapod_description/meshes/thigh_link.STL

Commit message: fix(climb): 更新左转移轨迹与关节限位
- 调整左后/左前摆动阶段位姿曲线、时长与着陆锚点
- 新增 quintic_first_segment 支持，使位姿在第一段提前完成
- 扩展部分髋关节限位并同步模板校验哈希

File: src/grasp_hexapod_description/urdf/grasp_hexapod.urdf (robot description, URDF)
Before this commit: robot grasp_hexapod, 19 links, 18 joints
Joints:
- joint lb_thigh_joint: limit lower=-0.698 upper=1.571 effort=1.2 velocity=4 -> lower=-1.047065850398866 upper=1.571 effort=1.2 velocity=4
- joint lf_thigh_joint: limit lower=-1.571 upper=0.698 effort=1.2 velocity=4 -> lower=-1.571 upper=1.047065850398866 effort=1.2 velocity=4
- joint rb_thigh_joint: limit lower=-1.571 upper=0.698 effort=1.2 velocity=4 -> lower=-1.571 upper=1.047065850398866 effort=1.2 velocity=4
- joint rf_thigh_joint: limit lower=-0.698 upper=1.571 effort=1.2 velocity=4 -> lower=-1.047065850398866 upper=1.571 effort=1.2 velocity=4

File: src/grasp_hexapod_description/urdf/hexapod_collision.urdf (robot description, URDF)
Before this commit: robot hexapod_robot, 25 links, 24 joints
Joints:
- joint lb_thigh_joint: limit lower=-0.698 upper=1.571 effort=1.2 velocity=4.0 -> lower=-1.047065850398866 upper=1.571 effort=1.2 velocity=4.0
- joint lf_thigh_joint: limit lower=-1.571 upper=0.698 effort=1.2 velocity=4.0 -> lower=-1.571 upper=1.047065850398866 effort=1.2 velocity=4.0
- joint rb_thigh_joint: limit lower=-1.571 upper=0.698 effort=1.2 velocity=4.0 -> lower=-1.571 upper=1.047065850398866 effort=1.2 velocity=4.0
- joint rf_thigh_joint: limit lower=-0.698 upper=1.571 effort=1.2 velocity=4.0 -> lower=-1.047065850398866 upper=1.571 effort=1.2 velocity=4.0

File: src/grasp_hexapod_description/urdf/hexapod_isaacgym_view.urdf (robot description, URDF)
Before this commit: robot hexapod_robot, 25 links, 24 joints
Joints:
- joint lb_thigh_joint: limit lower=-0.698 upper=1.571 effort=1.2 velocity=4.0 -> lower=-1.047065850398866 upper=1.571 effort=1.2 velocity=4.0
- joint lf_thigh_joint: limit lower=-1.571 upper=0.698 effort=1.2 velocity=4.0 -> lower=-1.571 upper=1.047065850398866 effort=1.2 velocity=4.0
- joint rb_thigh_joint: limit lower=-1.571 upper=0.698 effort=1.2 velocity=4.0 -> lower=-1.571 upper=1.047065850398866 effort=1.2 velocity=4.0
- joint rf_thigh_joint: limit lower=-0.698 upper=1.571 effort=1.2 velocity=4.0 -> lower=-1.047065850398866 upper=1.571 effort=1.2 velocity=4.0
